File: Power Distribution 2023-2024.kicad_sch (KiCad schematic)
At the start: 20 parts, among them J1 SAFETY_OUT, J2 STEER_OUT, J3 TEL_OUT, J4 E-STOP, J5 E-STOP, J6 E-STOP, J7 E-STOP

Commit message: November 11th, 2023 12:41pm
Parts:
- removed J7: E-STOP, Connector_Molex:Molex_Micro-Fit_3.0_43650-0200_1x02_P3.00mm_Horizontal, symbol Connector:Conn_01x02_Socket
- F1, F2, F3: footprint (none) -> Fuse:Fuseholder_Blade_Mini_Keystone_3568
- F4: renamed from F; footprint (none) -> Fuse:Fuseholder_Blade_Mini_Keystone_3568
- J1, J2: footprint Connector_Molex:Molex_Mega-Fit_76825-0004_2x02_P5.70mm_Horizontal -> Connector_Molex:Molex_Micro-Fit_3.0_43650-0200_1x02_P3.00mm_Horizontal
- renumbered D to D4, J to J4, J4 to J5, J5 to J6, J6 to J7, R to R4
Connections:
- net GND: now also J7.2 (Pin_2)
Other:
- moved on the sheet: D3, D4, F4, J3, J4, R3, R4

Commit message: November 11th, 2nd commit
Parts:
- J4: footprint Connector_Molex:Molex_Mega-Fit_76825-0004_2x02_P5.70mm_Horizontal -> FCP_Power_Distribution_Custom_Footprints:Molex_MegaFit_20024_1x02_P5.70mm_Horizontal
Changed lines of the file:
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@@
       (effects (font (size 1.27 1.27)) (justify left))
     )
-    (property "Footprint" "Connector_Molex:Molex_Mega-Fit_76825-0004_2x02_P5.70mm_Horizontal" (at 100.33 40.64 0)
+    (property "Footprint" "FCP_Power_Distribution_Custom_Footprints:Molex_MegaFit_20024_1x02_P5.70mm_Horizontal" (at 100.33 40.64 0)
       (effects (font (size 1.27 1.27)) hide)
     )

Commit message: PCB edits
Parts:
- added D5: LED, LED_SMD:LED_0805_2012Metric, symbol Device:LED
- added F5: Fuse, Fuse:Fuseholder_Blade_Mini_Keystone_3568, symbol Device:Fuse
- added He1, He2, He3, He4: MountingHole, MountingHole:MountingHole_2.7mm_M2.5_Pad, symbol Mechanical:MountingHole
- added R5: 4.7kΩ, Resistor_SMD:R_0805_2012Metric, symbol Device:R_US
Connections:
- net +12V: now also F5.1; no longer J5.1 (Pin_1)
- new net: F5.2, R5.1
- new net: D5.2 (A), R5.2
- new net: D5.1 (K), J5.1 (Pin_1)
Other:
- moved on the sheet: J5, J6, J7
