File: Power Distribution 2023-2024.kicad_sch (KiCad schematic)
At the start: 22 parts, among them J1 TEL_OUT, J2 STEER_OUT, J3 SAF_OUT, J4 12V_IN, J5 L_KILL, J6 R_KILL, J7 SAF_KILL

Commit message: November 25th, 2023
Parts:
- J3: value SAF_OUT -> SAFE_OUT
- J7: value SAF_KILL -> SAFE_KILL
Changed lines of the file:
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@@
   (paper "A4")
   (title_block
-    (date "2023-11-04")
+    (date "2023-11-25")
   )
   (junction (at 87.63 40.64) (diameter 0) (color 0 0 0 0)
@@
       (effects (font (size 1.27 1.27)) (justify left))
     )
-    (property "Value" "SAF_OUT" (at 252.73 46.99 0)
+    (property "Value" "SAFE_OUT" (at 252.73 46.99 0)
       (effects (font (size 1.27 1.27)) (justify left))
     )
@@
       (effects (font (size 1.27 1.27)) (justify left))
     )
-    (property "Value" "SAF_KILL" (at 245.11 93.98 0)
-      (effects (font (size 1.27 1.27)) (justify left))
-    )
+    (property "Value" "SAFE_KILL" (at 245.11 93.98 0)
+      (effects (font (size 1.27 1.27)) (justify left))
+    )
