File: Power Distribution 2023-2024.kicad_sch (KiCad schematic)
At the start: 22 parts, among them J1 TEL_OUT, J2 STEER_OUT, J3 SAFE_OUT, J4 12V_IN, J5 L_KILL, J6 R_KILL, J7 SAFE_KILL

Commit message: Schematic
Parts:
- removed D1, D2, D3, D5: LED, LED_SMD:LED_0805_2012Metric, symbol Device:LED
- removed F2, F3, F5: Fuse, Fuse:Fuseholder_Blade_Mini_Keystone_3568, symbol Device:Fuse
- removed J2: STEER_OUT, Connector_Molex:Molex_Micro-Fit_3.0_43650-0200_1x02_P3.00mm_Horizontal, symbol Connector:Conn_01x02_Socket
- removed J3: SAFE_OUT, Connector_Molex:Molex_Micro-Fit_3.0_43650-0200_1x02_P3.00mm_Horizontal, symbol Connector:Conn_01x02_Socket
- removed R1, R2, R3, R5: 4.7kΩ, Resistor_SMD:R_0805_2012Metric, symbol Device:R_US
- added J5: Conn_01x08_Shielded, Connector_RJ:RJ45_Amphenol_RJHSE5380, symbol Connector_Generic_Shielded:Conn_01x08_Shielded
- added J7: TURBO, Connector_Molex:Molex_Mini-Fit_Jr_5569-02A2_2x01_P4.20mm_Horizontal, symbol Connector:Conn_01x02_Socket
- J2: renamed from J5; value L_KILL -> EX_KILL
- J3: renamed from J7; value SAFE_KILL -> SAFETY
- J6: value R_KILL -> HORN; footprint Connector_Molex:Molex_Micro-Fit_3.0_43650-0200_1x02_P3.00mm_Horizontal -> Connector_Molex:Molex_Mini-Fit_Jr_5569-02A2_2x01_P4.20mm_Horizontal
Connections:
- net +12V: now also F4.1, R4.2, J5.1 (Pin_1), J5.2 (Pin_2); no longer F4.2, J4.1 (Pin_1)
- net GND: now also J6.1 (Pin_1), J5.SH (Shield), J7.1 (Pin_1)
- net at F1.2: now also J1.1 (Pin_1)
- net at J2.2 (Pin_2): now also J3.1 (Pin_1); no longer J6.1 (Pin_1)
- net HORN_OUT: now reaches J6.2 (Pin_2)
- net HORN_OUT: now also J5.6 (Pin_6); no longer J3.1 (Pin_1)
- net DRIVE_KILL: now reaches J2.1 (Pin_1)
- net DRIVE_KILL: now also J5.8 (Pin_8)
- new net: F4.2, J4.1 (Pin_1)
- new net TURBO_OUT: J5.7 (Pin_7), J7.2 (Pin_2)
- no-connect marks 0 -> 3
Other:
- note added: "12V"
- note added: "DRIVER INPUTS (from Steering Board)"
- note removed: "SAFETY"
- moved on the sheet: F1, J2, J3
