File: Power Distribution 2023-2024.kicad_pcb (KiCad board)
At the start: 2 copper layers, 19 parts, among them J1 SAFETY_OUT, J2 STEER_OUT, J3 TEL_OUT, J4 12V_IN, J5 E-STOP, J6 E-STOP, J7 E-STOP

Commit message: PCB edits
Parts:
- added D5: LED, LED_SMD:LED_0805_2012Metric, F.Cu at (224.2, 109.9)
- added F5: Fuse, Fuse:Fuseholder_Blade_Mini_Keystone_3568, F.Cu at (229.4, 124.3)
- added He1: MountingHole, MountingHole:MountingHole_2.7mm_M2.5_Pad, F.Cu at (216.5, 147.3)
- added He2: MountingHole, MountingHole:MountingHole_2.7mm_M2.5_Pad, F.Cu at (181.6, 129.5)
- added He3: MountingHole, MountingHole:MountingHole_2.7mm_M2.5_Pad, F.Cu at (174.0, 138.4)
- added He4: MountingHole, MountingHole:MountingHole_2.7mm_M2.5_Pad, F.Cu at (180.3, 152.4)
- added R5: 4.7kΩ, Resistor_SMD:R_0805_2012Metric, F.Cu at (228.6, 109.9)
- moved F1 149.6 mm to (245.3, 124.3), turned to 90 degrees
- moved F3 147.5 mm to (237.1, 124.3), turned to 90 degrees
- moved J3 144.5 mm to (254.8, 109.6), turned to -90 degrees
- moved F2 134.2 mm to (221.8, 124.3), turned to 90 degrees
- moved J2 133.5 mm to (222.9, 135.7), turned to 90 degrees
- moved J4 126.8 mm to (246.0, 133.3), turned to 90 degrees
- moved F4 124.4 mm to (228.1, 129.7), turned to 0 degrees
- moved D1 123.2 mm to (252.1, 119.4), turned to 90 degrees
- moved D3 119.9 mm to (250.8, 109.9), turned to 180 degrees
- moved R1 119.9 mm to (252.1, 115.3)
- moved J1 115.0 mm to (255.0, 120.3), turned to -90 degrees
- moved R3 111.7 mm to (247.0, 109.9)
- moved D4 110.1 mm to (236.6, 136.5), turned to 180 degrees
- moved J5 102.1 mm to (223.5, 107.0)
- moved J7 101.6 mm to (246.4, 107.0)
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Connections:
- J5 pad 1: +12V -> Net-(D5-K)
Routing:
- net GND: track 0.00 -> 79.0 mm
- net +12V: track 0.00 -> 44.8 mm
- net Net-(F2-Pad2): track 0.00 -> 12.7 mm
- net Net-(F3-Pad2): track 0.00 -> 12.4 mm
- net Net-(D2-K): track 0.00 -> 9.72 mm
- net Net-(J6-Pin_2): track 0.00 -> 9.06 mm
- net Net-(F4-Pad1): track 0.00 -> 8.08 mm
- net Net-(F1-Pad2): track 0.00 -> 8.01 mm
- net Net-(F5-Pad2): track 0.00 -> 8.00 mm
- net Net-(J5-Pin_2): track 0.00 -> 7.80 mm
- net Net-(D3-K): track 0.00 -> 3.09 mm
- net Net-(D5-K): track 0.00 -> 2.99 mm
- net Net-(D1-K): track 0.00 -> 2.94 mm
- net Net-(D4-A): track 0.00 -> 2.59 mm
- net Net-(D5-A): track 0.00 -> 2.51 mm
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- added copper zone on F.Cu, net +12V
- added copper zone on B.Cu, net GND
Other:
- board outline added: 50.8 x 52.7 mm

Commit message: November 25th, 2023
Parts:
- added G***: LOGO, FCP_Power_Distribution_Custom_Footprints:sm_logo, F.Cu at (248.9, 149.9)
- added REF**: GND, TestPoint:TestPoint_Keystone_5019_Minature, F.Cu at (237.4, 144.6)
- added REF**: 12V, TestPoint:TestPoint_Keystone_5019_Minature, F.Cu at (231.4, 144.6)
- J1: value SAFETY_OUT -> TEL_OUT
- J3: value TEL_OUT -> SAFE_OUT
- J5: value E-STOP -> L_KILL
- J6: value E-STOP -> R_KILL
- J7: value E-STOP -> SAFE_KILL
- moved He3 94.7 mm to (261.0, 100.9)
- moved He4 80.7 mm to (261.0, 149.9)
- moved He2 45.1 mm to (216.5, 100.9)
- moved J2 6.07 mm to (222.5, 141.8)
- moved D4 5.22 mm to (236.5, 141.7)
- moved R4 5.22 mm to (232.0, 141.7)
- moved D2 4.85 mm to (217.4, 131.7)
- moved R2 4.85 mm to (217.4, 127.9)
- moved F1 3.43 mm to (243.4, 127.2)
- moved D1 3.41 mm to (250.4, 122.3)
- moved R1 3.41 mm to (250.4, 118.2)
- moved F2 3.12 mm to (220.6, 127.2)
- moved F3 3.12 mm to (235.8, 127.2)
- moved F5 3.12 mm to (228.2, 127.2)
- moved J1 2.94 mm to (255.0, 123.2)
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Routing:
- net GND: track 79.0 -> 12.4 mm
- net +12V: track 44.8 -> 0.20 mm
- net Net-(F5-Pad2): track 8.00 -> 11.5 mm
- net Net-(D3-K): track 3.09 -> 5.76 mm
- net Net-(F4-Pad1): track 8.08 -> 10.7 mm
- net Net-(F2-Pad2): track 12.7 -> 14.5 mm
- net Net-(D1-K): track 2.94 -> 4.65 mm
- net Net-(F3-Pad2): track 12.4 -> 14.0 mm
- net Net-(D2-K): track 9.72 -> 11.2 mm
- net Net-(D5-K): track 2.99 -> 4.24 mm
- net Net-(F1-Pad2): track 8.01 -> 7.10 mm
- net Net-(D5-A): track 2.51 -> 1.72 mm
Other:
- board size 50.8 x 52.7 mm -> 50.8 x 55.2 mm
- board text added: "FCP Power Distribution 2025 Tomaz Zlindra"
- board text added: "F_12V_IN"
- board text added: "F_KILL"
- board text added: "F_SAF"
- board text added: "F_STEER"
- board text added: "F_TEL"
