File: Power Distribution 2023-2024.kicad_pcb (KiCad board)
At the start: 2 copper layers, 53.3 x 55.2 mm, 29 parts, among them J1 TEL_OUT, J2 STEER_OUT, J3 SAFE_OUT, J4 12V_IN, J5 L_KILL, J6 R_KILL, J7 SAFE_KILL

Commit message: December 2nd, 2023
Other:
- board text added: "FCP POWER SEMA 2025"
- board text added: "Sarah Qadar (lol)"
- board text added: "Tomaz Zlindra"
- board text removed: "FCP POWER SEMA 2025 Tomaz Zlindra Sarah Qadar"
Changed lines of the file:
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@@
   (gr_rect (start 213.36 97.79) (end 266.7 153.035)
     (stroke (width 0.1) (type default)) (fill none) (layer "Edge.Cuts"))
-  (gr_text "FCP POWER\nSEMA 2025\nTomaz Zlindra\nSarah Qadar" (at 226.06 152.4) (layer "F.SilkS")
-    (effects (font (size 1.5 1.5) (thickness 0.225)) (justify left bottom))
+  (gr_text "FCP POWER\nSEMA 2025\n" (at 226.452733 148.762235) (layer "F.SilkS")
+    (effects (font (size 1.75 1.75) (thickness 0.3) bold) (justify left bottom))
   )
   (gr_text "F_STEER" (at 219.772096 113.856974) (layer "F.SilkS")
@@
     (effects (font (size 1 1) (thickness 0.15)) (justify left bottom))
   )
+  (gr_text "Tomaz Zlindra" (at 226.50624 150.581461) (layer "F.SilkS")
+    (effects (font (size 1 1) (thickness 0.15)) (justify left bottom))
+  )
+  (gr_text "Sarah Qadar (lol)" (at 226.709884 151.557309) (layer "F.SilkS")
+    (effects (font (size 0.5 0.5) (thickness 0.1)) (justify left bottom))
+  )
   (gr_text "F_KILL" (at 228.569116 113.848962) (layer "F.SilkS")

Commit message: small error
Other:
- board text added: "Tomaz Zlindra Sarah Qadar"
- board text removed: "Sarah Qadar (lol)"
- board text removed: "Tomaz Zlindra"
Changed lines of the file:
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@@
     (effects (font (size 1 1) (thickness 0.15)) (justify left bottom))
   )
-  (gr_text "Tomaz Zlindra" (at 226.50624 150.581461) (layer "F.SilkS")
+  (gr_text "Tomaz Zlindra\nSarah Qadar" (at 226.535677 151.902819) (layer "F.SilkS")
     (effects (font (size 1 1) (thickness 0.15)) (justify left bottom))
-  )
-  (gr_text "Sarah Qadar (lol)" (at 226.709884 151.557309) (layer "F.SilkS")
-    (effects (font (size 0.5 0.5) (thickness 0.1)) (justify left bottom))
   )
   (gr_text "F_KILL" (at 228.569116 113.848962) (layer "F.SilkS")
@@
   (segment (start 249.896167 111.090103) (end 249.9 111.08627) (width 0.25) (layer "F.Cu") (net 6))
   (segment (start 246.348619 141.847267) (end 237.929634 141.847267) (width 2) (layer "F.Cu") (net 7))
-  (segment (start 257.804605 145.683068) (end 257.804605 149.86) (width 0.25) (layer "F.Cu") (net 7))
-  (segment (start 254.010225 141.888688) (end 257.804605 145.683068) (width 0.25) (layer "F.Cu") (net 7))
+  (segment (start 249.420693 141.888688) (end 253.645402 141.888688) (width 2) (layer "F.Cu") (net 7))
+  (segment (start 257.807261 146.050547) (end 257.804605 146.053203) (width 2) (layer "F.Cu") (net 7))
   (segment (start 246.39004 141.888688) (end 246.348619 141.847267) (width 2) (layer "F.Cu") (net 7))
   (segment (start 237.929634 141.847267) (end 236.497424 140.415057) (width 2) (layer "F.Cu") (net 7))
-  (segment (start 249.420693 141.888688) (end 254.010225 141.888688) (width 0.25) (layer "F.Cu") (net 7))
+  (segment (start 257.804605 146.053203) (end 257.804605 149.86) (width 2) (layer "F.Cu") (net 7))
+  (segment (start 253.645402 141.888688) (end 257.807261 146.050547) (width 2) (layer "F.Cu") (net 7))
   (segment (start 249.420693 141.888688) (end 246.39004 141.888688) (width 2) (layer "F.Cu") (net 7))
   (segment (start 232.945896 140.415057) (end 232.919645 140.388806) (width 0.25) (layer "F.Cu") (net 8))

Commit message: cleaned up stuff
Parts:
- moved G*** 15.2 mm to (234.0, 147.0)
- moved R5 2.24 mm to (226.0, 110.6), turned to 90 degrees
- moved REF** 1.85 mm to (224.0, 149.5)
- moved REF** 1.80 mm to (256.0, 149.9)
- moved F4 1.72 mm to (229.0, 133.8)
- moved D4 1.66 mm to (236.1, 142.0)
- moved R4 1.66 mm to (232.5, 142.0)
- moved D5 1.12 mm to (223.5, 111.0), turned to -90 degrees
- moved J4 0.75 mm to (248.7, 136.2)
- moved F2 0.73 mm to (220.6, 126.5)
- moved F3 0.73 mm to (235.8, 126.5)
- moved F5 0.73 mm to (228.2, 126.5)
- moved F1 0.73 mm to (243.4, 126.5)
Routing:
- net GND: track 27.5 -> 22.9 mm
- net Net-(F3-Pad2): track 15.5 -> 13.4 mm
- net Net-(D5-A): track 1.72 -> 3.44 mm
- net Net-(F5-Pad2): track 10.8 -> 9.54 mm
- net Net-(D5-K): track 4.73 -> 3.73 mm
- net Net-(D3-K): track 6.61 -> 7.53 mm
- net Net-(F2-Pad2): track 14.7 -> 15.5 mm
Other:
- board text added: "FCP POWER"
- board text added: "SEMA 2025"
- board text removed: "FCP POWER SEMA 2025"

Commit message: FINAL for printing (unless there are any last changes)
Other:
- board text added: "12V_IN"
- board text added: "KILL"
- board text added: "SAFETY"
- board text added: "STEER"
- board text added: "TEL"
- board text removed: "F_12V_IN"
- board text removed: "F_KILL"
- board text removed: "F_SAF"
- board text removed: "F_STEER"
- board text removed: "F_TEL"

Commit message: FINAL final final final
Parts:
- moved J4 0.75 mm to (249.4, 136.3)
Changed lines of the file:
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@@
   )
   (footprint "FCP_Power_Distribution_Custom_Footprints:Molex_MegaFit_20024_1x02_P5.70mm_Horizontal" (layer "F.Cu")
-    (at 248.670001 136.188687 90)
+    (at 249.414056 136.256176 90)
     (tags "2002411212 ")
     (property "Sheetfile" "Power Distribution 2023-2024.kicad_sch")
@@
   (segment (start 248.199393 111.090103) (end 249.896167 111.090103) (width 0.25) (layer "F.Cu") (net 6))
   (segment (start 249.896167 111.090103) (end 249.9 111.08627) (width 0.25) (layer "F.Cu") (net 6))
-  (segment (start 248.558689 142) (end 236.997424 142) (width 2) (layer "F.Cu") (net 7))
-  (segment (start 256.36 149.86) (end 248.670001 142.170001) (width 2) (layer "F.Cu") (net 7))
-  (segment (start 248.670001 142.170001) (end 248.670001 141.888688) (width 2) (layer "F.Cu") (net 7))
-  (segment (start 248.670001 141.888688) (end 248.558689 142) (width 2) (layer "F.Cu") (net 7))
+  (segment (start 236.997424 142) (end 249.370233 142) (width 2) (layer "F.Cu") (net 7))
+  (segment (start 256 149.86) (end 256 148.542121) (width 2) (layer "F.Cu") (net 7))
+  (segment (start 256 148.542121) (end 249.414056 141.956177) (width 2) (layer "F.Cu") (net 7))
+  (segment (start 249.370233 142) (end 249.414056 141.956177) (width 2) (layer "F.Cu") (net 7))
   (segment (start 235.446184 142) (end 233.553816 142) (width 0.25) (layer "F.Cu") (net 8))
   (segment (start 243.415749 116.5) (end 246.815749 116.5) (width 2) (layer "F.Cu") (net 10))

Commit message: DONE
Parts:
- removed D1, D2, D3, D5: LED, LED_SMD:LED_0805_2012Metric
- removed F2, F3, F5: Fuse, Fuse:Fuseholder_Blade_Mini_Keystone_3568
- removed the J2 at (222.5, 141.8)
- removed the J3 at (257.6, 113.0)
- removed R1, R2, R3, R5: 4.7kΩ, Resistor_SMD:R_0805_2012Metric
- added J5: Conn_01x08_Shielded, Connector_RJ:RJ45_Amphenol_RJHSE5380, F.Cu at (221.5, 126.8)
- added J7: TURBO, Connector_Molex:Molex_Mini-Fit_Jr_5569-02A2_2x01_P4.20mm_Horizontal, F.Cu at (227.4, 143.5)
- J2: renamed from J5; value L_KILL -> EX_KILL
- J3: renamed from J7; value SAFE_KILL -> SAFETY
- J6: value R_KILL -> HORN; footprint Connector_Molex:Molex_Micro-Fit_3.0_43650-0200_1x02_P3.00mm_Horizontal -> Connector_Molex:Molex_Mini-Fit_Jr_5569-02A2_2x01_P4.20mm_Horizontal
- moved REF** 52.1 mm to (222.6, 109.8)
- moved G*** 40.7 mm to (250.6, 109.8)
- moved J2 31.0 mm to (254.1, 117.3), turned to -90 degrees
- moved J6 30.8 mm to (227.3, 136.4), turned to 90 degrees
- moved J3 22.7 mm to (254.1, 128.6), turned to -90 degrees
- moved F4 21.6 mm to (242.1, 116.6), turned to -90 degrees
- moved R4 19.2 mm to (235.6, 123.0), turned to 90 degrees
- moved J1 16.1 mm to (254.1, 140.0)
- moved D4 15.4 mm to (235.6, 126.6), turned to 90 degrees
- moved F1 11.7 mm to (249.8, 116.7), turned to -90 degrees
- moved He3 9.49 mm to (260.0, 109.8)
- moved He2 9.10 mm to (216.3, 110.0)
- moved He4 3.49 mm to (260.0, 149.8)
- moved J4 2.71 mm to (247.1, 134.8), turned to 0 degrees
Connections:
- F1 pad 2: Net-(F1-Pad2) -> Net-(J1-Pin_1)
- F4 pad 1: Net-(F4-Pad1) -> +12V
- F4 pad 2: +12V -> Net-(J4-Pin_1)
- J1 pad 1: Net-(D1-K) -> Net-(J1-Pin_1)
- J2 pad 1: Net-(D5-K) -> /DRIVE_KILL
- J2 pad 2: Net-(J5-Pin_2) -> Net-(J2-Pin_2)
- J3 pad 1: Net-(J6-Pin_2) -> Net-(J2-Pin_2)
- J4 pad 1: +12V -> Net-(J4-Pin_1)
- J6 pad 1: Net-(J5-Pin_2) -> GND
- J6 pad 2: Net-(J6-Pin_2) -> /HORN_IN
- R4 pad 2: Net-(F4-Pad1) -> +12V
Routing:
- net /TURBO_IN: track 0.00 -> 35.1 mm
- net /DRIVE_KILL: track 0.00 -> 34.8 mm
- net /HORN_IN: track 0.00 -> 19.0 mm
- net Net-(J1-Pin_1): track 0.00 -> 18.6 mm
- net Net-(F2-Pad2): track 15.5 -> 0.00 mm
- net Net-(D2-K): track 15.2 -> 0.00 mm
- net Net-(J4-Pin_1): track 0.00 -> 13.7 mm
- net Net-(F3-Pad2): track 13.4 -> 0.00 mm
- net Net-(F1-Pad2): track 10.3 -> 0.00 mm
- net Net-(F4-Pad1): track 9.68 -> 0.00 mm
- net Net-(F5-Pad2): track 9.54 -> 0.00 mm
- net Net-(J5-Pin_2): track 8.48 -> 0.00 mm
- net Net-(J2-Pin_2): track 0.00 -> 8.36 mm
- net Net-(J6-Pin_2): track 8.36 -> 0.00 mm
- net GND: track 23.1 -> 15.2 mm
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Other:
- board size 53.3 x 55.2 mm -> 50 x 46.4 mm
- board text added: "12V"
- board text added: "EXTERNAL_KILL"
- board text added: "HORN"
- board text added: "J5"
- board text added: "SAFE_OUT"
- board text added: "STEER_OUT"
- board text added: "TURBO"
- board text removed: "12V_IN"
- board text removed: "KILL"
- board text removed: "SAFETY"
- board text removed: "STEER"
